File: hardware/kicad/NavPoTS.kicad_pcb (KiCad board)
At the start: 4 copper layers, 60 x 110 mm, 223 parts, among them J1 Screw_Terminal_01x02, J10 Screw_Terminal_01x02, J11 Screw_Terminal_01x06, J12 Screw_Terminal_01x06, J13 Screw_Terminal_01x02, J14 Screw_Terminal_01x02, J15 Conn_01x03_Pin, J16 Conn_01x03_Pin, J17 Conn_01x03_Pin, J18 Conn_01x03_Pin, J19 USB_C_Receptacle_USB2.0_16P, J2 Screw_Terminal_01x02, J20 Conn_01x03_Pin, J21 Conn_01x03_Pin, J22 Conn_01x03_Pin, J23 Conn_01x03_Pin, J3 DM3CS-SF, J4 Conn_Coaxial, J5 Conn_Coaxial, J6 Screw_Terminal_01x02, J7 Screw_Terminal_01x06, J8 Screw_Terminal_01x06, J9 Screw_Terminal_01x02, Q1 SI4143DY-T1-GE3, Q10 SI4143DY-T1-GE3, Q11 Q_NMOS_GSD, Q12 Q_NMOS_GSD, Q13 AO4576, Q14 AO4576, Q15 Q_NMOS_GSD, Q16 AO4576, Q17 AO4576, Q2 SI4143DY-T1-GE3, Q3 Q_NMOS_GSD, Q4 Q_NMOS_GSD, Q5 Q_NMOS_GSD, Q6 Q_NMOS_GSD, Q7 Q_NMOS_GSD, Q8 Q_NMOS_GSD, Q9 Q_NMOS_GSD, U1 MMC5983MA, U10 NEO-M8N, U11 AP64501SP-13, U12 INA226, U13 USBLC6-2SC6, U14 STM32H743ZITx, U2 MS5611-01BA, U3 H3LIS331DLTR, U4 SIC431A, U5 ASM330LHHXTR, U6 AP64501SP-13, U7 MB85RS2MTAPNF-G-BDERE1, U8 LTC4412xS6, U9 E22-900M33S, Y1 ECS-2520MV-xxx-xx

Commit message: sorted components into rough placement on pcb
Parts:
- moved U7 203.4 mm to (47.8, 157.8)
- moved Q16 185.0 mm to (70.8, 154.0)
- moved U9 178.6 mm to (37.9, 124.4)
- moved J3 177.1 mm to (71.4, 183.2)
- moved Q13 161.7 mm to (84.5, 40.9)
- moved Q10 149.4 mm to (100.5, 29.1)
- moved C43 147.3 mm to (242.0, 74.8)
- moved C44 147.3 mm to (242.0, 77.8)
- moved C45 147.3 mm to (242.0, 80.8)
- moved C47 139.9 mm to (251.6, 68.8)
- moved Q14 136.6 mm to (115.0, 42.4)
- moved Q17 135.9 mm to (124.7, 159.1)
- moved Y1 135.8 mm to (57.8, 86.3)
- moved F1 132.4 mm to (79.0, 45.8)
- moved C40 130.0 mm to (236.9, 66.2)
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Other:
- board size 60 x 110 mm -> 44 x 100 mm
