File: hardware/kicad/NavPoTS-Bridge/NavPoTS-Bridge.kicad_pcb (KiCad board)
At the start: 4 copper layers, 58.9 x 58.9 mm, 74 parts, among them J1 Conn_01x06_Pin, J2 USB_C_Receptacle_USB2.0_16P, J3 Screw_Terminal_01x06, J4 Conn_02x04_Top_Bottom, J5 Conn_02x04_Top_Bottom, J6 Conn_02x04_Top_Bottom, J7 62684-402100ALF, J8 62684-402100ALF, J9 Conn_02x04_Top_Bottom, U1 MS5611-01BA, U2 H3LIS331DLTR, U3 ASM330LHHXTR, U4 MMC5983MA, U5 USBLC6-2SC6, U6 STM32H743ZITx, Y1 ECS-2520MV-xxx-xx

Commit message: v1.0
Connections:
- J7 pad 10: SPI2_CS3 -> GNSS_nRST
- J7 pad 11: GNSS_nRST -> SPI2_CS3
- U6 pad 80: SPI2_CS3 -> GNSS_nRST
- U6 pad 81: GNSS_nRST -> SPI2_CS3
Other:
- board text added: "v1.0 - 6/13/26 Luke Hooper"
Changed lines of the file:
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@@
 			(plot_on_all_layers_selection 0x00000000_00000000_00000000_00000000)
 			(disableapertmacros no)
-			(usegerberextensions no)
+			(usegerberextensions yes)
 			(usegerberattributes yes)
 			(usegerberadvancedattributes yes)
-			(creategerberjobfile yes)
+			(creategerberjobfile no)
 			(dashed_line_dash_ratio 12.000000)
 			(dashed_line_gap_ratio 3.000000)
@@
 			(outputformat 1)
 			(mirror no)
-			(drillshape 1)
+			(drillshape 0)
 			(scaleselection 1)
-			(outputdirectory "")
+			(outputdirectory "/home/Luke/cad/kicad/projects/NavPoTS-R1/Bridge/gerbers/")
 		)
 	)
@@
 			(size 0.3 1.2)
 			(layers "F.Cu" "F.Mask" "F.Paste")
-			(net 52 "SPI2_CS3")
+			(net 66 "GNSS_nRST")
 			(pinfunction "10")
 			(pintype "passive")
@@
 			(size 0.3 1.2)
 			(layers "F.Cu" "F.Mask" "F.Paste")
-			(net 66 "GNSS_nRST")
+			(net 52 "SPI2_CS3")
 			(pinfunction "11")
 			(pintype "passive")
@@
 			(layers "F.Cu" "F.Mask" "F.Paste")
 			(roundrect_rratio 0.25)
-			(net 52 "SPI2_CS3")
+			(net 66 "GNSS_nRST")
 			(pinfunction "PD11")
 			(pintype "bidirectional")
@@
 			(layers "F.Cu" "F.Mask" "F.Paste")
 			(roundrect_rratio 0.25)
-			(net 66 "GNSS_nRST")
+			(net 52 "SPI2_CS3")
 			(pinfunction "PD12")
 			(pintype "bidirectional")
@@
 			)
 		)
+		(property "MPN" "PEC14SAGN"
+			(at 0 0 180)
+			(unlocked yes)
+			(layer "B.Fab")
+			(hide yes)
+			(effects
+				(font
+					(size 1 1)
+					(thickness 0.15)
+				)
+				(justify mirror)
+			)
+		)
+		(property "Manufacturer" "Sullins Connector Solutions"
+			(at 0 0 180)
+			(unlocked yes)
+			(layer "B.Fab")
+			(hide yes)
+			(effects
+				(font
+					(size 1 1)
+					(thickness 0.15)
+				)
+				(justify mirror)
+			)
+		)
 		(property ki_fp_filters "Connector*:*_2x??_*")
 		(sheetname "/")
@@
 			)
 		)
+		(property "MPN" "PEC14SAGN"
+			(at 0 0 0)
+			(unlocked yes)
+			(layer "B.Fab")
+			(hide yes)
+			(effects
+				(font
+					(size 1 1)
+					(thickness 0.15)
+				)
+				(justify mirror)
+			)
+		)
+		(property "Manufacturer" "Sullins Connector Solutions"
+			(at 0 0 0)
+			(unlocked yes)
+			(layer "B.Fab")
+			(hide yes)
+			(effects
+				(font
+					(size 1 1)
+					(thickness 0.15)
+				)
+				(justify mirror)
+			)
+		)
 		(property ki_fp_filters "Connector*:*_2x??_*")
 		(sheetname "/")
@@
 			)
 		)
+		(property "MPN" "PEC14SAGN"
+			(at 0 0 0)
+			(unlocked yes)
+			(layer "B.Fab")
+			(hide yes)
+			(effects
+				(font
+					(size 1 1)
+					(thickness 0.15)
+				)
+				(justify mirror)
+			)
+		)
+		(property "Manufacturer" "Sullins Connector Solutions"
+			(at 0 0 0)
+			(unlocked yes)
+			(layer "B.Fab")
+			(hide yes)
+			(effects
+				(font
+					(size 1 1)
+					(thickness 0.15)
+				)
+				(justify mirror)
+			)
+		)
 		(property ki_fp_filters "Connector*:*_2x??_*")
 		(sheetname "/")
@@
 			)
 		)
+		(property "MPN" "PEC14SAGN"
+			(at 0 0 180)
+			(unlocked yes)
+			(layer "B.Fab")
+			(hide yes)
+			(effects
+				(font
+					(size 1 1)
+					(thickness 0.15)
+				)
+				(justify mirror)
+			)
+		)
+		(property "Manufacturer" "Sullins Connector Solutions"
+			(at 0 0 180)
+			(unlocked yes)
+			(layer "B.Fab")
+			(hide yes)
+			(effects
+				(font
+					(size 1 1)
+					(thickness 0.15)
+				)
+				(justify mirror)
+			)
+		)
 		(property ki_fp_filters "Connector*:*_2x??_*")
 		(sheetname "/")
@@
 		(layer "Edge.Cuts")
 	)
+	(gr_text "v1.0 - 6/13/26\nLuke Hooper"
+		(at 190.75 91.25 0)
+		(layer "B.SilkS")
+		(effects
+			(font
+				(size 1 1)
+				(thickness 0.15)
+			)
+			(justify left bottom mirror)
+		)
+	)
 	(segment
 		(start 189.3875 86.8625)
@@
 	)
 	(segment
-		(start 210.662489 105.250011)
-		(end 218.424989 105.250011)
+		(start 210.662489 104.750011)
+		(end 218.424989 104.750011)
 		(width 0.2)
 		(layer "F.Cu")
@@
 	)
 	(segment
-		(start 218.424989 105.250011)
-		(end 218.425 105.25)
+		(start 218.424989 104.750011)
+		(end 218.425 104.75)
 		(width 0.2)
 		(layer "F.Cu")
@@
 	)
 	(segment
-		(start 210.662489 104.750011)
-		(end 218.424989 104.750011)
+		(start 210.662489 105.250011)
+		(end 218.424989 105.250011)
 		(width 0.2)
 		(layer "F.Cu")
@@
 	)
 	(segment
-		(start 218.424989 104.750011)
-		(end 218.425 104.75)
+		(start 218.424989 105.250011)
+		(end 218.425 105.25)
 		(width 0.2)
 		(layer "F.Cu")
