File: hardware/kicad/NavPoTS-Bridge/NavPoTS-Bridge.kicad_pcb (KiCad board)
At the start: 4 copper layers, 58.9 x 58.9 mm, 74 parts, among them J1 Conn_01x06_Pin, J2 USB_C_Receptacle_USB2.0_16P, J3 Screw_Terminal_01x06, J4 Conn_02x04_Top_Bottom, J5 Conn_02x04_Top_Bottom, J6 Conn_02x04_Top_Bottom, J7 62684-402100ALF, J8 62684-402100ALF, J9 Conn_02x04_Top_Bottom, U1 MS5611-01BA, U2 H3LIS331DLTR, U3 ASM330LHHXTR, U4 MMC5983MA, U5 USBLC6-2SC6, U6 STM32H743ZITx, Y1 ECS-2520MV-xxx-xx

Commit message: correct zener diode placement to be on rx instead of tx for usart_3
Parts:
- moved R13 0.41 mm to (205.0, 119.9)
Connections:
- D2 pad 1: USART3_TX -> USART3_RX
- J3 pad 6: USART3_RX -> USART3_TX
- R13 pad 1: USART3_TX -> USART3_RX
Routing:
- net USART3_TX: track 8.98 -> 16.6 mm, vias 0 -> 1
- net USART3_RX: track 15.1 -> 9.60 mm
- net GND: track 145.5 -> 145.3 mm, vias 76 -> 77
Changed lines of the file:
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@@
 	(footprint "Resistor_SMD:R_0603_1608Metric_Pad0.98x0.95mm_HandSolder"
 		(layer "F.Cu")
-		(at 205 119.5 -90)
+		(at 205 119.912511 -90)
 		(descr "Resistor SMD 0603 (1608 Metric), square (rectangular) end terminal, IPC-7351 nominal with elongated pad for handsoldering. (Body size source: IPC-SM-782 page 72, https://www.pcb-3d.com/wordpress/wp-content/uploads/ipc-sm-782a_amendment_1_and_2.pdf)")
 		(tags "resistor handsolder")
@@
 			(layers "F.Cu" "F.Mask" "F.Paste")
 			(roundrect_rratio 0.25)
-			(net "USART3_TX")
+			(net "USART3_RX")
 			(pintype "passive")
 		)
@@
 			(layers "F.Cu" "F.Mask" "F.Paste")
 			(roundrect_rratio 0.25)
-			(net "USART3_TX")
+			(net "USART3_RX")
 			(pinfunction "K_1")
 			(pintype "passive")
@@
 			(layers "*.Cu" "*.Mask")
 			(remove_unused_layers no)
-			(net "USART3_RX")
+			(net "USART3_TX")
 			(pinfunction "Pin_6_6")
 			(pintype "passive")
@@
 	)
 	(segment
-		(start 208.15 116.5)
-		(end 206.75 116.5)
-		(width 0.3)
-		(layer "F.Cu")
-		(net "GND")
-	)
-	(segment
 		(start 203.249989 112.249989)
 		(end 203.25 112.25)
@@
 	)
 	(segment
+		(start 208.15 116.5)
+		(end 207 116.5)
+		(width 0.3)
+		(layer "F.Cu")
+		(net "GND")
+	)
+	(segment
 		(start 198.249989 111.915369)
 		(end 198.294187 111.959567)
@@
 	)
 	(segment
+		(start 207 116.5)
+		(end 206.999989 116.500011)
+		(width 0.3)
+		(layer "F.Cu")
+		(net "GND")
+	)
+	(segment
 		(start 204.32 75.43)
 		(end 204.25 75.5)
@@
 	)
 	(via
-		(at 206.75 116.5)
+		(at 200 85.25)
 		(size 0.6)
 		(drill 0.3)
@@
 	)
 	(via
-		(at 200 85.25)
+		(at 216.15 90.75)
 		(size 0.6)
 		(drill 0.3)
@@
 	)
 	(via
-		(at 216.15 90.75)
+		(at 203.499989 120.500011)
+		(size 0.6)
+		(drill 0.3)
+		(layers "F.Cu" "B.Cu")
+		(net "GND")
+	)
+	(via
+		(at 206.999989 116.500011)
 		(size 0.6)
 		(drill 0.3)
 		(layers "F.Cu" "B.Cu")
-		(capping no)
-		(covering
-			(front no)
-			(back no)
-		)
-		(plugging
-			(front no)
-			(back no)
-		)
-		(filling no)
 		(net "GND")
 	)
@@
 	)
 	(segment
-		(start 207.249989 112.500011)
-		(end 204.85 114.9)
+		(start 207.249989 112.151459)
+		(end 206.950713 112.450735)
 		(width 0.2)
 		(layer "F.Cu")
@@
 	)
 	(segment
-		(start 207.249989 110.662511)
-		(end 207.249989 112.500011)
+		(start 209 124.5)
+		(end 208.5 125)
 		(width 0.2)
 		(layer "F.Cu")
@@
 	)
 	(segment
-		(start 205 116.65)
-		(end 204.85 116.5)
+		(start 207.249989 110.662511)
+		(end 207.249989 112.151459)
 		(width 0.2)
 		(layer "F.Cu")
 		(net "USART3_TX")
 	)
+	(via
+		(at 206.950713 112.450735)
+		(size 0.6)
+		(drill 0.3)
+		(layers "F.Cu" "B.Cu")
+		(net "USART3_TX")
+	)
 	(segment
-		(start 205 118.5875)
-		(end 205 116.65)
+		(start 206.950713 112.450735)
+		(end 205.999989 113.401459)
 		(width 0.2)
-		(layer "F.Cu")
+		(layer "B.Cu")
 		(net "USART3_TX")
 	)
 	(segment
-		(start 204.85 114.9)
-		(end 204.85 116.5)
+		(start 205.999989 113.401459)
+		(end 205.999989 122.499989)
 		(width 0.2)
-		(layer "F.Cu")
+		(layer "B.Cu")
+		(net "USART3_TX")
+	)
+	(segment
+		(start 205.999989 122.499989)
+		(end 208.5 125)
+		(width 0.2)
+		(layer "B.Cu")
 		(net "USART3_TX")
 	)
 	(segment
-		(start 204.999999 125)
-		(end 205 120.4125)
+		(start 205 120.825011)
+		(end 204.999999 125)
 		(width 0.2)
 		(layer "F.Cu")
@@
 	)
 	(segment
-		(start 209 124.5)
-		(end 208.5 125)
+		(start 205 119.000011)
+		(end 205 116.65)
 		(width 0.2)
 		(layer "F.Cu")
@@
 	)
 	(segment
-		(start 209 113.75)
-		(end 209 124.5)
+		(start 205 116.65)
+		(end 204.85 116.5)
 		(width 0.2)
 		(layer "F.Cu")
@@
 	(segment
 		(start 207.749989 112.499989)
-		(end 209 113.75)
+		(end 204.85 115.399978)
+		(width 0.2)
+		(layer "F.Cu")
+		(net "USART3_RX")
+	)
+	(segment
+		(start 204.85 115.399978)
+		(end 204.85 116.5)
 		(width 0.2)
 		(layer "F.Cu")
