File: hardware/kicad/NavPoTS-North/NavPoTS-North.kicad_sch (KiCad schematic)
At the start: 44 parts, among them J3 DM3CS-SF, J4 Conn_Coaxial, J5 Conn_Coaxial, Q11 Q_NMOS_GSD, Q12 Q_NMOS_GSD, Q15 Q_NMOS_GSD, Q5 Q_NMOS_GSD, U10 NEO-M8N, U7 MB85RS2MTAPNF-G-BDERE1, U9 E22-900M33S

Commit message: remaped pins and renamed pcb sections
Parts:
- renumbered C30 to C1, C23 to C10, C31 to C2, C32 to C3, C39 to C4, C27 to C5, C28 to C6, C29 to C7, C24 to C8, C25 to C9, D2 to D1, D5 to D2, D6 to D3, D8 to D4, D7 to D5, H9 to H1, H10 to H2, H11 to H3, H12 to H4, J5 to J1, J4 to J2, L3 to L1, Q5 to Q1, Q11 to Q2, Q15 to Q3, Q12 to Q4, R24 to R1, R42 to R10, R38 to R11, R14 to R12, R23 to R13, R21 to R14, R25 to R2, R26 to R3, R27 to R4, R36 to R5, R37 to R6, R17 to R7, R18 to R8, R33 to R9, U10 to U1, U9 to U2, U7 to U3
Other:
- title: (none) -> NavPoTS-North

Commit message: finished first draft of north pcb routing
Parts:
- removed R9: 10k, Resistor_SMD:R_0603_1608Metric_Pad0.98x0.95mm_HandSolder, symbol Device:R
- added J10, J4, J6, J8: Conn_02x04_Top_Bottom, Connector_PinSocket_2.54mm:PinSocket_2x04_P2.54mm_Vertical, symbol Connector_Generic:Conn_02x04_Top_Bottom
- added J5, J9: Conn_01x02, Connector_JST:JST_XH_B2B-XH-A_1x02_P2.50mm_Vertical, symbol Connector_Generic:Conn_01x02
- added J7: 62684-402100ALF, custom:Amphenol_62684-402100ALF, symbol custom:62684-402100ALF
- added Q1, Q4: Q_NMOS_GSD, Package_TO_SOT_SMD:SOT-23-3, symbol Transistor_FET:Q_NMOS_GSD
- U3: renamed from U1; footprint RF_GPS:ublox_NEO -> custom:NEO-M8N
- renumbered C8 to C1, C4 to C10, C9 to C2, C5 to C3, C6 to C4, C7 to C5, C10 to C6, C1 to C7, C2 to C8, C3 to C9, J3 to J1, J1 to J3, Q1 to Q2, Q2 to Q3, Q3 to Q5, Q4 to Q6, R12 to R1, R5 to R10, R6 to R11, R10 to R12, R11 to R13, R7 to R2, R8 to R3, R13 to R4, R14 to R5, R1 to R6, R2 to R7, R3 to R8, R4 to R9, U3 to U1
Connections:
- net +3V3: now also J10.1 (Pin_1), J10.2 (Pin_2), J10.3 (Pin_3), J10.4 (Pin_4), J4.1 (Pin_1), J4.2 (Pin_2), J4.3 (Pin_3), J4.4 (Pin_4), J5.1 (Pin_1), J6.1 (Pin_1), J6.2 (Pin_2), J6.3 (Pin_3), J6.4 (Pin_4), J8.1 (Pin_1), J8.2 (Pin_2), J8.3 (Pin_3), J8.4 (Pin_4), J9.1 (Pin_1)
- net DEBUG_2: now also J7.18
- net DEBUG_3: now also J7.19
- net DEBUG_4: now also J7.20
- net DEBUG_5: now also J7.21
- net GND: now also J10.5 (Pin_5), J10.6 (Pin_6), J10.7 (Pin_7), J10.8 (Pin_8), J4.5 (Pin_5), J4.6 (Pin_6), J4.7 (Pin_7), J4.8 (Pin_8), J6.5 (Pin_5), J6.6 (Pin_6), J6.7 (Pin_7), J6.8 (Pin_8), J7.S1 (SHIELD), J7.S2 (SHIELD), J8.5 (Pin_5), J8.6 (Pin_6), J8.7 (Pin_7), J8.8 (Pin_8), Q1.2 (S), Q4.2 (S)
- net GNSS_nRST: now also J7.10
- net LoRa_BUSY: now also J7.15
- net LoRa_IO: now also J7.16
- net LoRa_RXEN: now also J7.12
- net LoRa_nRST: now also J7.17
- net SPI2_CS0: now also J7.07
- net SPI2_CS1: now also J7.08
- net SPI2_CS2: now also J7.09
- net SPI2_CS3: now also J7.11
- net SPI2_MISO: now also J7.05
- net SPI2_MOSI: now also J7.06
- net SPI2_SCK: now also J7.04
- new net: J5.2 (Pin_2), Q1.3 (D)
- new net: J9.2 (Pin_2), Q4.3 (D)
- new net EXT_PWR2: J7.26, Q1.1 (G)
- new net EXT_PWR3: J7.27, Q4.1 (G)
- new net GPIO_7: J7.28
- new net GPIO_8: J7.29
- new net GPIO_9: J7.30
- no-connect marks 7 -> 26
Other:
- note added: "BRIDGE BOARD"
- note added: "IO"
- moved on the sheet: C1, C10, C2, C3, C4, C5, C6, C7, C8, C9, D1, D2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

Commit message: v1.0
Parts:
- J10, J4, J6, J8: MPN (none) -> 61300821821; Manufacturer (none) -> Würth Elektronik
- U3: footprint custom:NEO-M8N -> RF_GPS:ublox_NEO
Changed lines of the file:
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@@
 			)
 		)
-		(property "Footprint" "custom:NEO-M8N"
+		(property "Footprint" "RF_GPS:ublox_NEO"
 			(at 271.78 86.36 0)
 			(effects
@@
 			)
 		)
+		(property "MPN" "61300821821"
+			(at 50.8 167.64 0)
+			(effects
+				(font
+					(size 1.27 1.27)
+				)
+				(hide yes)
+			)
+		)
+		(property "Manufacturer" "Würth Elektronik"
+			(at 50.8 167.64 0)
+			(effects
+				(font
+					(size 1.27 1.27)
+				)
+				(hide yes)
+			)
+		)
 		(pin "8"
 		)
@@
 			)
 		)
+		(property "MPN" "61300821821"
+			(at 49.53 123.19 0)
+			(effects
+				(font
+					(size 1.27 1.27)
+				)
+				(hide yes)
+			)
+		)
+		(property "Manufacturer" "Würth Elektronik"
+			(at 49.53 123.19 0)
+			(effects
+				(font
+					(size 1.27 1.27)
+				)
+				(hide yes)
+			)
+		)
 		(pin "8"
 		)
@@
 			)
 		)
+		(property "MPN" "61300821821"
+			(at 49.53 146.05 0)
+			(effects
+				(font
+					(size 1.27 1.27)
+				)
+				(hide yes)
+			)
+		)
+		(property "Manufacturer" "Würth Elektronik"
+			(at 49.53 146.05 0)
+			(effects
+				(font
+					(size 1.27 1.27)
+				)
+				(hide yes)
+			)
+		)
 		(pin "8"
 		)
@@
 			(at 49.53 100.33 0)
 			(effects
+				(font
+					(size 1.27 1.27)
+				)
+				(hide yes)
+			)
+		)
+		(property "MPN" "61300821821"
+			(at 49.53 100.33 0)
+			(effects
+				(font
+					(size 1.27 1.27)
+				)
+				(hide yes)
+			)
+		)
+		(property "Manufacturer" "Würth Elektronik"
+			(at 49.53 100.33 0)
+			(effects

Commit message: update to kicad, begin cad work for pcb holder bracket
Parts:
- D2, D3, D4, D5: footprint LED_SMD:LED_PLCC_2835_Handsoldering -> custom:LED_PLCC_2835_Handsoldering
- U3: footprint RF_GPS:ublox_NEO -> custom:NEO-M8N
