File: hardware/kicad/NavPoTS-South/NavPoTS-South.kicad_sch (KiCad schematic)
At the start: 118 parts, among them J1 Screw_Terminal_01x02, J10 Screw_Terminal_01x02, J13 Screw_Terminal_01x02, J14 Screw_Terminal_01x02, J15 Conn_01x03_Pin, J16 Conn_01x03_Pin, J17 Conn_01x03_Pin, J18 Conn_01x03_Pin, J2 Screw_Terminal_01x02, J20 Conn_01x03_Pin, J21 Conn_01x03_Pin, J22 Conn_01x03_Pin, J23 Conn_01x03_Pin, J6 Screw_Terminal_01x02, J7 Screw_Terminal_01x06, J8 Screw_Terminal_01x06, J9 Screw_Terminal_01x02, Q1 SI4143DY-T1-GE3, Q10 SI4143DY-T1-GE3, Q13 AO4576, Q14 AO4576, Q16 AO4576, Q17 AO4576, Q2 SI4143DY-T1-GE3, Q3 Q_NMOS_GSD, Q4 Q_NMOS_GSD, Q6 Q_NMOS_GSD, Q7 Q_NMOS_GSD, Q8 Q_NMOS_GSD, Q9 Q_NMOS_GSD, U11 AP64501SP-13, U12 INA226, U4 SIC431A, U6 AP64501SP-13, U8 LTC4412xS6

Commit message: remaped pins and renamed pcb sections
Parts:
- added J11, J12, J3, J5: Conn_02x04_Top_Bottom, Connector_PinSocket_2.54mm:PinSocket_2x04_P2.54mm_Vertical, symbol Connector_Generic:Conn_02x04_Top_Bottom
- added J4: 62684-402100ALF, custom:Amphenol_62684-402100ALF, symbol custom:62684-402100ALF
Connections:
- net +3V3: now also J11.1 (Pin_1), J11.2 (Pin_2), J11.3 (Pin_3), J11.4 (Pin_4), J12.1 (Pin_1), J12.2 (Pin_2), J12.3 (Pin_3), J12.4 (Pin_4), J3.1 (Pin_1), J3.2 (Pin_2), J3.3 (Pin_3), J3.4 (Pin_4), J5.1 (Pin_1), J5.2 (Pin_2), J5.3 (Pin_3), J5.4 (Pin_4)
- net EXT_PWR0: now also J4.04
- net EXT_PWR1: now also J4.05
- net EXT_PWR2: now also J4.06
- net EXT_PWR3: now also J4.17
- net EXT_PWR4: now also J4.18
- net EXT_PWR5: now also J4.19
- net GND: now also J11.5 (Pin_5), J11.6 (Pin_6), J11.7 (Pin_7), J11.8 (Pin_8), J12.5 (Pin_5), J12.6 (Pin_6), J12.7 (Pin_7), J12.8 (Pin_8), J3.5 (Pin_5), J3.6 (Pin_6), J3.7 (Pin_7), J3.8 (Pin_8), J4.S1 (SHIELD), J4.S2 (SHIELD), J5.5 (Pin_5), J5.6 (Pin_6), J5.7 (Pin_7), J5.8 (Pin_8)
- net I2C1_SCL: now also J4.08
- net I2C1_SDA: now also J4.07
- net PGOOD: now also J4.02
- net PWM_0: now also J4.20
- net PWM_1: now also J4.21
- net PWM_2: now also J4.22
- net PWM_3: now also J4.23
- net PWM_4: now also J4.24
- net PWM_5: now also J4.25
- net PWM_6: now also J4.26
- net PWM_7: now also J4.27
- net PYRO0_CONTINUITY: now also J4.10
- net PYRO0_FIRE: now also J4.09
- net PYRO1_CONTINUITY: now also J4.12
- net PYRO1_FIRE: now also J4.11
- net PYRO2_CONTINUITY: now also J4.14
- net PYRO2_FIRE: now also J4.13
- net PYRO3_CONTINUITY: now also J4.16
- net PYRO3_FIRE: now also J4.15
- net VSTAT: now also J4.03
- net V_ALERT: now also J4.01
- no-connect marks 4 -> 16
Other:
- note added: "SOUTH BOARD"
- title: (none) -> NavPoTS-South
- moved on the sheet: D10, D13, D14, D3, D9, F1, F2, F3, F4, H5, H6, H7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

Commit message: first draft of south board layout and high current traces
Parts:
- removed D3: RED, LED_SMD:LED_PLCC_2835_Handsoldering, symbol Device:LED
- removed J4: 62684-402100ALF, custom:Amphenol_62684-402100ALF, symbol custom:62684-402100ALF
- removed J7, J8: Screw_Terminal_01x06, custom:CONN_ED555_6DS, symbol Connector:Screw_Terminal_01x06
- removed Q7, Q9: Q_NMOS_GSD, Package_TO_SOT_SMD:SOT-23-3, symbol Transistor_FET:Q_NMOS_GSD
- removed R34: 100R, Resistor_SMD:R_0603_1608Metric_Pad0.98x0.95mm_HandSolder, symbol Device:R
- added D2: RED, LED_SMD:LED_0603_1608Metric_Pad1.05x0.95mm_HandSolder, symbol Device:D
- added J1, J5: Screw_Terminal_01x02, custom:CONN_ED555_2DS, symbol Connector:Screw_Terminal_01x02
- added J23: 62684-402100ALF, custom:Amphenol_62684-402100ALF, symbol custom:62684-402100ALF
- added J3, J6, J7, J8: Conn_01x02, Connector_JST:JST_XH_B2B-XH-A_1x02_P2.50mm_Vertical, symbol Connector_Generic:Conn_01x02
- added Q2, Q8: Q_NMOS_GSD, Package_TO_SOT_SMD:SOT-23-3, symbol Transistor_FET:Q_NMOS_GSD
- added R21: 220R, Resistor_SMD:R_0603_1608Metric_Pad0.98x0.95mm_HandSolder, symbol Device:R
- Q4: now not fitted; now left out of the parts list
- Q6: renamed from Q8; now not fitted; now left out of the parts list
- renumbered C6 to C1, C19 to C10, C20 to C11, C21 to C12, C22 to C13, C26 to C14, C33 to C15, C34 to C16, C35 to C17, C36 to C18, C37 to C19, C7 to C2, C38 to C20, C40 to C21, C41 to C22, C42 to C23, C43 to C24, C44 to C25, C45 to C26, C46 to C27, C47 to C28, C8 to C3, C12 to C4, C14 to C5, C15 to C6, C16 to C7, C17 to C8, C18 to C9, D9 to D3, D10 to D4, D13 to D5, D14 to D6, H5 to H1, H6 to H2, H7 to H3, H8 to H4, J16 to J10, J17 to J11, J18 to J12, J20 to J13, J21 to J14, J22 to J15, J23 to J16, J6 to J17, J11 to J18, J3 to J19, J1 to J2, J9 to J20, J10 to J21, J5 to J22, J12 to J24, J13 to J25, J14 to J26, J2 to J4, J15 to J9, L4 to L3, Q3 to Q1, Q13 to Q10, Q14 to Q11, Q16 to Q12, Q17 to Q13, Q6 to Q3, Q1 to Q5, Q2 to Q7, Q10 to Q9, R15 to R10, R16 to R11, R19 to R12, R20 to R13, R22 to R14, R28 to R15, R29 to R16, R30 to R17, R31 to R18, R32 to R19, R4 to R2, R33 to R20, R40 to R22, R41 to R23, R43 to R24, R44 to R25, R45 to R26, R46 to R27, R50 to R28, R51 to R29, R6 to R3, R55 to R30, R56 to R31, R59 to R32, R60 to R33, R63 to R34, R64 to R35, R65 to R36, R66 to R37, R7 to R4, R9 to R5, R10 to R6, R11 to R7, R12 to R8, R13 to R9, U4 to U1, U6 to U2, U8 to U3, U11 to U4, U12 to U5
Connections:
- net +3V3: now also J3.1 (Pin_1)
- net +5V: now also J1.1 (Pin_1), J5.1 (Pin_1), J6.1 (Pin_1), J7.1 (Pin_1), J8.1 (Pin_1)
- net EXT_PWR0: now also J23.06
- net EXT_PWR1: now also J23.07
- net EXT_PWR2: now also J23.09
- net EXT_PWR3: now also J23.28, Q2.1 (G); no longer Q4.1 (G)
- net EXT_PWR4: now also Q4.1 (G), J23.29
- net EXT_PWR5: now also J23.30, Q8.1 (G)
- net GND: now also J23.S1 (SHIELD), J23.S2 (SHIELD), Q2.2 (S), Q8.2 (S), R21.2
- net I2C1_SCL: now also J23.13
- net I2C1_SDA: now also J23.12
- net PGOOD: now also J23.04
- net PWM_0: now also J23.31
- net PWM_1: now also J23.32
- net PWM_2: now also J23.33
- net PWM_3: now also J23.34
- net PWM_4: now also J23.35
- net PWM_5: now also J23.36
- net PWM_6: now also J23.37
- net PWM_7: now also J23.38
- net PYRO0_CONTINUITY: now also J23.15
- net PYRO0_FIRE: now also J23.14
- net PYRO1_CONTINUITY: now also J23.17
- net PYRO1_FIRE: now also J23.16
- net PYRO2_CONTINUITY: now also J23.21
- net PYRO2_FIRE: now also J23.20
- net PYRO3_CONTINUITY: now also J23.23
- net PYRO3_FIRE: now also J23.22
- net PYRO_HIGH_SIDE: now also D2.2 (A)
- net VSTAT: now also J23.05
- net V_ALERT: now also J23.03
- net at Q1.3 (D): now also J1.2 (Pin_2)
- net at Q3.3 (D): now also J5.2 (Pin_2)
- net at Q6.3 (D): now also J7.2 (Pin_2)
- net at Q4.3 (D): now also J6.2 (Pin_2)
- new net: J8.2 (Pin_2), Q8.3 (D)
- new net: D2.1 (K), R21.1
- new net: J3.2 (Pin_2), Q2.3 (D)
Other:
- moved on the sheet: J10, J11, J12, J13, J14, J15, J16, J9, Q1, Q3

Commit message: first draft of south board routing
Parts:
- removed J3, J6, J7, J8: Conn_01x02, Connector_JST:JST_XH_B2B-XH-A_1x02_P2.50mm_Vertical, symbol Connector_Generic:Conn_01x02
- removed Q2, Q4, Q6, Q8: Q_NMOS_GSD, Package_TO_SOT_SMD:SOT-23-3, symbol Transistor_FET:Q_NMOS_GSD
- renumbered J14 to J10, J15 to J11, J16 to J12, J17 to J13, J18 to J14, J19 to J15, J20 to J16, J21 to J17, J22 to J18, J23 to J19, J24 to J20, J25 to J21, J26 to J22, J4 to J3, J5 to J4, J9 to J5, J10 to J6, J11 to J7, J12 to J8, J13 to J9, Q3 to Q2, Q5 to Q3, Q7 to Q4, Q9 to Q5, Q10 to Q6, Q11 to Q7, Q12 to Q8, Q13 to Q9
Connections:
- net EXT_PWR4 is gone; now on net EXT_PWR1: J19.29
- net EXT_PWR5 is gone; now on net EXT_PWR0: J19.30
- net EXT_PWR0: no longer J19.06
- net EXT_PWR1: no longer J19.07
- net EXT_PWR2: no longer names the net of J19.09
- net EXT_PWR3: no longer names the net of J19.28
- no-connect marks 16 -> 20

Commit message: added gpio for future use on north and south boards
Parts:
- removed J19: 62684-402100ALF, custom:Amphenol_62684-402100ALF, symbol custom:62684-402100ALF
- added J18: 62684-402100ALF, custom:Amphenol_62684-402100ALF, symbol custom:62684-402100ALF
- renumbered J18 to J19
Connections:
- net EXT_PWR0: now also J18.30
- net EXT_PWR1: now also J18.29
- net GND: now also J18.S1 (SHIELD), J18.S2 (SHIELD)
- net I2C1_SCL: now also J18.13
- net I2C1_SDA: now also J18.12
- net PGOOD: now also J18.04
- net PWM_0: now also J18.31
- net PWM_1: now also J18.32
- net PWM_2: now also J18.33
- net PWM_3: now also J18.34
- net PWM_4: now also J18.35
- net PWM_5: now also J18.36
- net PWM_6: now also J18.37
- net PWM_7: now also J18.38
- net PYRO0_CONTINUITY: now also J18.15
- net PYRO0_FIRE: now also J18.14
- net PYRO1_CONTINUITY: now also J18.17
- net PYRO1_FIRE: now also J18.16
- net PYRO2_CONTINUITY: now also J18.21
- net PYRO2_FIRE: now also J18.20
- net PYRO3_CONTINUITY: now also J18.23
- net PYRO3_FIRE: now also J18.22
- net VSTAT: now also J18.05
- net V_ALERT: now also J18.03
- new net GPIO_0: J18.06
- new net GPIO_1: J18.07
- new net GPIO_2: J18.09
- new net GPIO_3: J18.10
- new net GPIO_4: J18.11
- new net GPIO_5: J18.24
- new net GPIO_6: J18.28
- no-connect marks 20 -> 13

Commit message: finished first draft of north pcb routing
Other:
- note added: "BRIDGE BOARD"
- note removed: "SOUTH BOARD"
Changed lines of the file:
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@@
 		)
 	)
-	(text "SOUTH BOARD"
+	(text "BRIDGE BOARD"
 		(exclude_from_sim no)
-		(at 201.676 218.186 0)
+		(at 202.184 218.186 0)
 		(effects
 			(font

Commit message: v1.0
Parts:
- added TP1, TP3, TP4: TestPoint, TestPoint:TestPoint_Pad_D1.5mm, symbol Connector:TestPoint
- J14, J15, J19, J20: MPN (none) -> 61300821821; Manufacturer (none) -> Würth Elektronik
- renumbered J2 to J1, J1 to J2, TP1 to TP2
Connections:
- net +3V3: now also TP4.1
- net +5V: now also TP3.1
- net +8V: now also TP1.1
Other:
- moved on the sheet: J10, J11, J12, J2, J4, J5, J6, J7, J8, J9, Q1, Q2

Commit message: update to kicad, begin cad work for pcb holder bracket
Parts:
- U5: footprint Package_SO:VSSOP-10_3x3mm_P0.5mm -> Package_SO:TSSOP-10_3x3mm_P0.5mm
